File: V1/Relay-24v-8ch-V1.kicad_pcb (KiCad board)
At the start: 2 copper layers, 108 x 67.8 mm, 49 parts, among them J1 Conn_01x09, J2 OUT1, J3 OUT2, J4 OUT3, J5 OUT4, J6 OUT5, J7 OUT6, J8 OUT7, J9 OUT8, K1 G5PZ-1A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

Commit message: Change connector 3D model
Parts:
- J1: footprint Tales:TerminalBlock_Dorabo_DB141V-2.54-09P_1x09_P2.54mm_Vertical -> Tales:TerminalBlock_DG141V-2.54-9P_1x09_P2.54mm_Vertical
- moved R8 34.9 mm to (162.2, 60.3)
- moved R1 28.8 mm to (129.9, 60.3), turned to 180 degrees
- moved D8 26.5 mm to (122.4, 64.8), turned to 0 degrees
- moved R7 22.5 mm to (162.2, 62.9)
- moved D7 19.6 mm to (117.3, 64.8), turned to 0 degrees
- moved R2 17.1 mm to (129.9, 62.9), turned to 180 degrees
- moved D16 16.3 mm to (184.9, 64.8)
- moved R4 15.0 mm to (129.9, 67.9), turned to 180 degrees
- moved D11 14.4 mm to (169.7, 64.8)
- moved D4 13.7 mm to (112.2, 64.8), turned to 0 degrees
- moved R6 11.4 mm to (162.2, 65.4)
- moved D15 11.4 mm to (179.9, 64.8)
- moved D12 10.5 mm to (174.8, 64.8)
- moved D3 10.3 mm to (107.2, 64.8), turned to 0 degrees
- moved R3 9.54 mm to (129.9, 65.4), turned to 180 degrees
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Routing:
- net +24V: track 186.4 -> 212.2 mm
- net Net-(D3-A): track 1.98 -> 24.4 mm
- net Net-(D16-A): track 1.98 -> 24.4 mm
- net Net-(D6-A): track 29.3 -> 51.6 mm, vias 0 -> 1
- net Net-(D5-A): track 38.0 -> 56.5 mm, vias 0 -> 1
- net Net-(D4-A): track 1.98 -> 18.0 mm
- net Net-(D15-A): track 1.99 -> 18.0 mm
- net Net-(D2-A): track 47.4 -> 60.5 mm, vias 0 -> 1
- net Net-(D11-K): track 29.3 -> 42.0 mm, vias 0 -> 1
- net Net-(D7-A): track 1.98 -> 12.2 mm
- net Net-(D12-A): track 1.98 -> 12.2 mm
- net Net-(D10-A): track 38.0 -> 47.9 mm, vias 0 -> 1
- net Net-(D13-A): track 47.4 -> 57.0 mm, vias 0 -> 1
- net Net-(D8-A): track 1.99 -> 7.11 mm
- net Net-(D11-A): track 1.99 -> 7.11 mm
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Other:
- board text added: "CONN PINOUT: +24V-OUT1...OUT8"

Commit message: Update silkscreen and board image.
Other:
- board text added: "+24V-IN1-IN2-...-IN8"
- board text added: "IN1"
- board text added: "IN2"
- board text added: "IN3"
- board text added: "IN4"
- board text added: "IN5"
- board text added: "IN6"
- board text added: "IN7"
- board text added: "IN8"
- board text added: "RELAY-24V-8CH-V1"
- board text added: "TMASCHIO 2023"
- board text removed: "CONN PINOUT: +24V-OUT1...OUT8"
Changed lines of the file:
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@@
   (gr_line (start 120.015 69.215) (end 120.015 63.5)
     (stroke (width 0.15) (type default)) (layer "F.SilkS"))
+  (gr_line (start 105.41 62.23) (end 124.46 62.23)
+    (stroke (width 0.15) (type default)) (layer "F.SilkS"))
+  (gr_line (start 132.08 59.055) (end 132.98 59.23)
+    (stroke (width 0.15) (type default)) (layer "F.SilkS"))
   (gr_line (start 187.325 69.215) (end 167.005 69.215)
+    (stroke (width 0.15) (type default)) (layer "F.SilkS"))
+  (gr_line (start 105.41 59.055) (end 105.41 62.23)
     (stroke (width 0.15) (type default)) (layer "F.SilkS"))
   (gr_line (start 124.46 120.015) (end 124.46 124.46)
@@
   (gr_line (start 162.56 120.015) (end 162.56 124.46)
     (stroke (width 0.35) (type solid)) (layer "F.SilkS"))
+  (gr_line (start 124.46 62.23) (end 124.46 59.055)
+    (stroke (width 0.15) (type default)) (layer "F.SilkS"))
+  (gr_line (start 105.41 59.055) (end 132.08 59.055)
+    (stroke (width 0.15) (type default)) (layer "F.SilkS"))
   (gr_line (start 172.72 120.015) (end 172.72 124.46)
     (stroke (width 0.35) (type solid)) (layer "F.SilkS"))
@@
     (effects (font (size 1.5 1.5) (thickness 0.25)))
   )
-  (gr_text "OUT3" (at 117.348 68.58) (layer "F.SilkS")
+  (gr_text "RELAY-24V-8CH-V1" (at 189.865 60.96) (layer "F.SilkS")
+    (effects (font (size 1.4 1) (thickness 0.15)))
+  )
+  (gr_text "IN3" (at 117.348 68.58) (layer "F.SilkS")
     (effects (font (size 1.8 1.2) (thickness 0.2)) (justify bottom))
+  )
+  (gr_text "TMASCHIO 2023" (at 173.99 60.96) (layer "F.SilkS")
+    (effects (font (size 1.4 1) (thickness 0.15)))
   )
   (gr_text "V~ LOAD" (at 167.64 121.285) (layer "F.SilkS")
     (effects (font (size 1.5 1.3) (thickness 0.2)))
   )
-  (gr_text "OUT5" (at 169.672 68.58) (layer "F.SilkS")
+  (gr_text "IN5" (at 169.672 68.58) (layer "F.SilkS")
     (effects (font (size 1.8 1.2) (thickness 0.2)) (justify bottom))
   )
@@
     (effects (font (size 1.5 1.3) (thickness 0.2)))
   )
-  (gr_text "CONN PINOUT: +24V-OUT1...OUT8" (at 97.79 61.595) (layer "F.SilkS")
+  (gr_text "+24V-IN1-IN2-...-IN8" (at 106.045 61.595) (layer "F.SilkS")
     (effects (font (size 1.5 1) (thickness 0.2)) (justify left bottom))
   )
-  (gr_text "OUT2" (at 112.268 68.58) (layer "F.SilkS")
+  (gr_text "IN2" (at 112.268 68.58) (layer "F.SilkS")
     (effects (font (size 1.8 1.2) (thickness 0.2)) (justify bottom))
   )
@@
     (effects (font (size 1.5 1.3) (thickness 0.2)))
   )
-  (gr_text "OUT8" (at 184.912 68.58) (layer "F.SilkS")
+  (gr_text "IN8" (at 184.912 68.58) (layer "F.SilkS")
     (effects (font (size 1.8 1.2) (thickness 0.2)) (justify bottom))
   )
-  (gr_text "OUT4" (at 122.428 68.58) (layer "F.SilkS")
+  (gr_text "IN4" (at 122.428 68.58) (layer "F.SilkS")
     (effects (font (size 1.8 1.2) (thickness 0.2)) (justify bottom))
   )
@@
     (effects (font (size 1.5 1.3) (thickness 0.2)))
   )
-  (gr_text "OUT6" (at 174.752 68.58) (layer "F.SilkS")
+  (gr_text "IN6" (at 174.752 68.58) (layer "F.SilkS")
     (effects (font (size 1.8 1.2) (thickness 0.2)) (justify bottom))
   )
-  (gr_text "OUT1" (at 107.188 68.58) (layer "F.SilkS")
+  (gr_text "IN1" (at 107.188 68.58) (layer "F.SilkS")
     (effects (font (size 1.8 1.2) (thickness 0.2)) (justify bottom))
   )
-  (gr_text "OUT7" (at 179.832 68.58) (layer "F.SilkS")
+  (gr_text "IN7" (at 179.832 68.58) (layer "F.SilkS")
     (effects (font (size 1.8 1.2) (thickness 0.2)) (justify bottom))
   )

Commit message: Update to silkscreen and board image.
Parts:
- moved J1 20.8 mm to (157.5, 62.9), turned to 180 degrees
- moved D11 2.54 mm to (172.2, 64.8)
- moved D15 2.54 mm to (182.4, 64.8)
- moved R5 2.54 mm to (164.7, 67.9)
- moved R6 2.54 mm to (164.7, 65.4)
- moved R7 2.54 mm to (164.7, 62.9)
- moved R8 2.54 mm to (164.7, 60.3)
- moved D3 2.54 mm to (109.7, 64.8)
- moved D12 2.54 mm to (177.3, 64.8)
- moved D16 2.54 mm to (187.5, 64.8)
- moved D4 2.54 mm to (114.8, 64.8)
- moved D7 2.54 mm to (119.9, 64.8)
- moved D8 2.54 mm to (124.9, 64.8)
- moved R1 2.54 mm to (132.4, 60.3)
- moved R2 2.54 mm to (132.4, 62.9)
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Connections:
- J1 pad 1: +24V -> Net-(D14-A)
- J1 pad 2: Net-(D1-A) -> Net-(D13-A)
- J1 pad 3: Net-(D2-A) -> Net-(D10-A)
- J1 pad 4: Net-(D5-A) -> Net-(D11-K)
- J1 pad 6: Net-(D11-K) -> Net-(D5-A)
- J1 pad 7: Net-(D10-A) -> Net-(D2-A)
- J1 pad 8: Net-(D13-A) -> Net-(D1-A)
- J1 pad 9: Net-(D14-A) -> +24V
Routing:
- net Net-(D6-A): track 51.6 -> 48.6 mm
- net Net-(D13-A): track 57.0 -> 54.6 mm
- net Net-(D5-A): track 56.5 -> 54.9 mm
- net Net-(D11-K): track 42.0 -> 43.5 mm
- net Net-(D10-A): track 47.9 -> 46.8 mm
- net +24V: track 212.2 -> 211.5 mm
- net Net-(D1-A): track 58.1 -> 57.4 mm
