File: V2/Relay-24v-8ch-V2.kicad_pcb (KiCad board)
At the start: 2 copper layers, 98 x 67.8 mm, 44 parts, among them J1 DB141V-2.54-6P, J2 DB141V-2.54-6P, J3 DB142V-5.08-8P, J4 DB142V-5.08-8P, K1 G5PZ-1A, K2 G5PZ-1A, K3 G5PZ-1A, K4 G5PZ-1A, K5 G5PZ-1A, K6 G5PZ-1A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

Commit message: Redone everything
Parts:
- K1, K2, K3, K4, K5, K6, K7, K8: value G5PZ-1A -> G5Q-1A4-DC24V; footprint Tales:Relay_SPST_Omron_G5PZ-1A -> Tales:Relay_SPST_Omron-G5Q-1A
Connections:
- K1 pad 2: Net-(J3-Pin_1) -> Net-(J3-Pin_2)
- K1 pad 3: Net-(J3-Pin_2) -> Net-(J3-Pin_1)
- K2 pad 2: Net-(J3-Pin_3) -> Net-(J3-Pin_4)
- K2 pad 3: Net-(J3-Pin_4) -> Net-(J3-Pin_3)
- K3 pad 2: Net-(J3-Pin_5) -> Net-(J3-Pin_6)
- K3 pad 3: Net-(J3-Pin_6) -> Net-(J3-Pin_5)
- K4 pad 2: Net-(J3-Pin_7) -> Net-(J3-Pin_8)
- K4 pad 3: Net-(J3-Pin_8) -> Net-(J3-Pin_7)
- K5 pad 2: Net-(J4-Pin_1) -> Net-(J4-Pin_2)
- K5 pad 3: Net-(J4-Pin_2) -> Net-(J4-Pin_1)
- K6 pad 2: Net-(J4-Pin_3) -> Net-(J4-Pin_4)
- K6 pad 3: Net-(J4-Pin_4) -> Net-(J4-Pin_3)
- K7 pad 2: Net-(J4-Pin_5) -> Net-(J4-Pin_6)
- K7 pad 3: Net-(J4-Pin_6) -> Net-(J4-Pin_5)
- K8 pad 2: Net-(J4-Pin_7) -> Net-(J4-Pin_8)
- K8 pad 3: Net-(J4-Pin_8) -> Net-(J4-Pin_7)
Routing:
- net Net-(J4-Pin_2): track 44.3 -> 66.2 mm
- net Net-(J3-Pin_2): track 44.3 -> 66.2 mm
- net Net-(J4-Pin_8): track 44.7 -> 66.6 mm
- net Net-(J4-Pin_4): track 42.9 -> 64.8 mm
- net Net-(J3-Pin_8): track 44.7 -> 66.6 mm
- net Net-(J3-Pin_6): track 43.2 -> 65.1 mm
- net Net-(J3-Pin_4): track 42.9 -> 64.8 mm
- net Net-(J4-Pin_6): track 43.2 -> 65.1 mm
Other:
- board text added: "MAX 8A PER CHANNEL 2023 TMASCHIO"
- board text added: "RELAY-24V-8CH-V2"
- board text removed: "MAX 12A PER CHANNEL 2023 TMASCHIO"
- board text removed: "RELAY-24V-8CH-V1"
