File: V2/Relay-24v-8ch-V2.kicad_sch (KiCad schematic)
At the start: 44 parts, among them J1 DB141V-2.54-6P, J2 DB141V-2.54-6P

Commit message: Redone everything
Parts:
- K? (x8): value G5PZ-1A -> G5Q-1A4-DC24V; footprint Tales:Relay_SPST_Omron_G5PZ-1A -> Tales:Relay_SPST_Omron-G5Q-1A; symbol Tales:G5PZ-1A -> Tales:G5Q-1A; JLCPCB BOM 0 -> 1; LCSC Part # (none) -> C2931104; Mfr Omron -> Omron Electronics; Mfr PN G5PZ-1A -> G5Q-1A4-DC24V; Vendor Mouser -> JLCPCB; Vendor PN 653-G5PZ-1ADC24 -> C2931104
Connections:
- net at D?.1 (K), D?.2 (A), J2.2 (Pin_2): now also K?.5; no longer K?.4
- net at J?.1 (Pin_1), RV?.1: now also K?.3; no longer K?.2 (x2)
- net at J?.2 (Pin_2), RV?.2: now also K?.2; no longer K?.3 (x2)
- net at D?.1 (K), D?.2 (A), J1.1 (Pin_1): now also K?.5; no longer K?.4
- net at J?.5 (Pin_5), RV?.1: now also K?.3; no longer K?.2 (x2)
- net at J?.6 (Pin_6), RV?.2: now also K?.2; no longer K?.3 (x2)
- net at D?.1 (K), D?.2 (A), J1.2 (Pin_2): now also K?.5; no longer K?.4
- net at D?.1 (K), D?.2 (A), J1.4 (Pin_4): now also K?.5; no longer K?.4
- net at D?.1 (K), D?.2 (A), J2.3 (Pin_3): now also K?.5; no longer K?.4
- net at D?.1 (K), D?.2 (A), J2.4 (Pin_4): now also K?.5; no longer K?.4
- net at J?.7 (Pin_7), RV?.1: now also K?.3; no longer K?.2 (x2)
- net at J?.8 (Pin_8), RV?.2: now also K?.2; no longer K?.3 (x2)
- net at D?.1 (K), D?.2 (A), J2.1 (Pin_1): now also K?.5; no longer K?.4
- net at J?.3 (Pin_3), RV?.1: now also K?.3; no longer K?.2 (x2)
- net at J?.4 (Pin_4), RV?.2: now also K?.2; no longer K?.3 (x2)
- net at D?.1 (K), D?.2 (A), J1.3 (Pin_3): now also K?.5; no longer K?.4
Other:
- moved on the sheet: D?, K?, R?, RV?
